Commit message: 现在的负载估计是真正在仿真环境中产生负载了！缺点是第一，负载在生成以后就无法再次随机，如果一定要在add_load中重新生成，会导致负载重置。这是比较底层的问题。第二，目前的负载基本还是一个一个生成。第三，需要注意在迭代几千步以后再开始生成负载。第四，注意现在extra_loss只有前7项，虽然有点浪费算力，但这无疑减少了不少工作量。

File: resources/robots/WF_TRON1A/urdf/robot_proto.urdf (robot description, URDF)
Before this commit: robot wheel_biped, 11 links, 10 joints
Links:
- removed link plate_link
Joints:
- removed joint plate_fixed_joint
