Commit message: 负载加载可能有问题版本

File: resources/robots/WF_TRON1A/urdf/robot.urdf (robot description, URDF)
Before this commit: robot wheel_biped, 10 links, 9 joints
Links:
- added link plate_link, mass 0.1; collision box size=0.5 0.5 0.005; visual box size=0.5 0.5 0.005
Joints:
- added joint plate_fixed_joint: type fixed, parent base_Link, child plate_link, origin xyz=0 0 0.02 rpy=0 0 0
